Commit message: ros2_control working with all the interfaces

File: ROS/src/asabe_robot_description/urdf/robot_description_arm.urdf (robot description, URDF)
Before this commit: robot asabe_robot_description, 5 links, 4 joints
Links:
- removed link Link_wheel1
- removed link Link_wheel2
- removed link Link_wheel3
- removed link Link_wheel4
- added link Link_arm1, mass 0.52977; collision mesh filename=package://asabe_robot_description/meshes/Link_arm1.STL; visual mesh filename=package://asabe_robot_description/meshes/Link_arm1.STL
- added link Link_arm2, mass 0.38055; collision mesh filename=package://asabe_robot_description/meshes/Link_arm2.STL; visual mesh filename=package://asabe_robot_description/meshes/Link_arm2.STL
- added link Link_arm3, mass 0.52829; collision mesh filename=package://asabe_robot_description/meshes/Link_arm3.STL; visual mesh filename=package://asabe_robot_description/meshes/Link_arm3.STL
- added link Link_arm4, mass 0.23793; collision mesh filename=package://asabe_robot_description/meshes/Link_arm4.STL; visual mesh filename=package://asabe_robot_description/meshes/Link_arm4.STL
- added link Link_arm5, mass 0.12412; collision mesh filename=package://asabe_robot_description/meshes/Link_arm5.STL; visual mesh filename=package://asabe_robot_description/meshes/Link_arm5.STL
- added link Link_arm6, mass 0.043811; collision mesh filename=package://asabe_robot_description/meshes/Link_arm6.STL; visual mesh filename=package://asabe_robot_description/meshes/Link_arm6.STL
- added link base, mass 0.78986; collision mesh filename=package://asabe_robot_description/meshes/base_link.STL; visual mesh filename=package://asabe_robot_description/meshes/base_link.STL
- added link grasp_point
- link base_link: mass 0.78986 -> None
Joints:
- removed joint Joint_wheel1
- removed joint Joint_wheel2
- removed joint Joint_wheel3
- removed joint Joint_wheel4
- added joint Joint_arm1: type fixed, parent base, child Link_arm1, origin xyz=-0.084 0 0 rpy=0 0 0, axis 0 0 0
- added joint Joint_arm2: type revolute, parent Link_arm1, child Link_arm2, origin xyz=0 0 0.035 rpy=0 0 0, axis 0 0 -1, limit lower=0 upper=5.0 effort=0 velocity=0.5
- added joint Joint_arm3: type prismatic, parent Link_arm2, child Link_arm3, origin xyz=0 0 0.0405 rpy=0 0 0, axis 0 0 1, limit lower=0 upper=0.18 effort=0 velocity=0.03
- added joint Joint_arm4: type revolute, parent Link_arm3, child Link_arm4, origin xyz=0 -0.0835 0.16784 rpy=-1.5708 0 0, axis 0 0 1, limit lower=0 upper=1.5708 effort=0 velocity=0.5
- added joint Joint_arm5: type prismatic, parent Link_arm4, child Link_arm5, origin xyz=0.0445 0 -0.031 rpy=0 -1.5708 0, axis 0 0 -1, limit lower=0 upper=0.1 effort=0 velocity=0.03
- added joint Joint_arm6: type fixed, parent Link_arm5, child Link_arm6, origin xyz=0.0094 0.0397 -0.12045 rpy=0 3.14159 3.14159, axis 0 0 1, limit lower=-3.14 upper=3.14 effort=0 velocity=0
- added joint Joint_base: type fixed, parent base_link, child base, origin xyz=0 0 0 rpy=0 0 0, axis 0 0 0
- added joint Joint_grasp_point: type fixed, parent Link_arm6, child grasp_point, origin xyz=0 0 0.1 rpy=3.14159 -1.5707 0, axis 0 0 0
