Commit message: gazebo world and urdf updated

File: ROS/src/asabe_robot_description/urdf/robot_description.urdf (robot description, URDF)
Before this commit: robot asabe_robot_description, 12 links, 11 joints
Links:
- removed link Link_arm1
- removed link Link_arm2
- removed link Link_arm3
- removed link Link_arm4
- removed link Link_arm5
- removed link Link_arm6
- removed link grasp_point
Joints:
- removed joint Joint_arm1
- removed joint Joint_arm2
- removed joint Joint_arm3
- removed joint Joint_arm4
- removed joint Joint_arm5
- removed joint Joint_arm6
- removed joint Joint_grasp_point

Commit message: ros2_control integration (all the controllers)

File: ROS/src/asabe_robot_description/urdf/robot_description.urdf (robot description, URDF)
Before this commit: robot asabe_robot_description, 5 links, 4 joints
Links:
- added link Link_arm1, mass 0.52977; collision mesh filename=package://asabe_robot_description/meshes/Link_arm1.STL; visual mesh filename=package://asabe_robot_description/meshes/Link_arm1.STL
- added link Link_arm2, mass 0.38055; collision mesh filename=package://asabe_robot_description/meshes/Link_arm2.STL; visual mesh filename=package://asabe_robot_description/meshes/Link_arm2.STL
- added link Link_arm3, mass 0.52829; collision mesh filename=package://asabe_robot_description/meshes/Link_arm3.STL; visual mesh filename=package://asabe_robot_description/meshes/Link_arm3.STL
- added link Link_arm4, mass 0.23793; collision mesh filename=package://asabe_robot_description/meshes/Link_arm4.STL; visual mesh filename=package://asabe_robot_description/meshes/Link_arm4.STL
- added link Link_arm5, mass 0.12412; collision mesh filename=package://asabe_robot_description/meshes/Link_arm5.STL; visual mesh filename=package://asabe_robot_description/meshes/Link_arm5.STL
- added link Link_arm6, mass 0.043811; collision mesh filename=package://asabe_robot_description/meshes/Link_arm6.STL; visual mesh filename=package://asabe_robot_description/meshes/Link_arm6.STL
- added link base, mass 0.78986; collision mesh filename=package://asabe_robot_description/meshes/base_link.STL; visual mesh filename=package://asabe_robot_description/meshes/base_link.STL
- added link grasp_point
- link base_link: mass 0.78986 -> None
Joints:
- added joint Joint_arm1: type fixed, parent base, child Link_arm1, origin xyz=-0.084 0 0 rpy=0 0 0, axis 0 0 0
- added joint Joint_arm2: type revolute, parent Link_arm1, child Link_arm2, origin xyz=0 0 0.035 rpy=0 0 0, axis 0 0 -1, limit lower=0 upper=5.0 effort=0 velocity=0.5
- added joint Joint_arm3: type prismatic, parent Link_arm2, child Link_arm3, origin xyz=0 0 0.0405 rpy=0 0 0, axis 0 0 1, limit lower=0 upper=0.18 effort=0 velocity=0.03
- added joint Joint_arm4: type revolute, parent Link_arm3, child Link_arm4, origin xyz=0 -0.0835 0.16784 rpy=-1.5708 0 0, axis 0 0 1, limit lower=0 upper=1.5708 effort=0 velocity=0.5
- added joint Joint_arm5: type prismatic, parent Link_arm4, child Link_arm5, origin xyz=0.0445 0 -0.031 rpy=0 -1.5708 0, axis 0 0 -1, limit lower=0 upper=0.1 effort=0 velocity=0.03
- added joint Joint_arm6: type fixed, parent Link_arm5, child Link_arm6, origin xyz=0.0094 0.0397 -0.12045 rpy=0 3.14159 3.14159, axis 0 0 1, limit lower=-3.14 upper=3.14 effort=0 velocity=0
- added joint Joint_base: type fixed, parent base_link, child base, origin xyz=0 0 0 rpy=0 0 0, axis 0 0 0
- added joint Joint_grasp_point: type fixed, parent Link_arm6, child grasp_point, origin xyz=0 0 0.1 rpy=3.14159 -1.5707 0, axis 0 0 0
- joint Joint_wheel4: limit lower=0 upper=0 effort=0 velocity=0 -> (none)

Commit message: footprint

File: ROS/src/asabe_robot_description/urdf/robot_description.urdf (robot description, URDF)
Before this commit: robot asabe_robot_description, 13 links, 12 joints
Links:
- added link base_footprint
- link base_link: geometry visual mesh filename=package://asabe_robot_description/meshes/base_link.STL
Joints:
- added joint base_joint: type fixed, parent base_link, child base_footprint, origin xyz=0.0 0.0 -0.01875 rpy=0 0 0

Commit message: Navigation working :')

File: ROS/src/asabe_robot_description/urdf/robot_description.urdf (robot description, URDF)
Before this commit: robot asabe_robot_description, 14 links, 13 joints
Links:
- removed link base_footprint
- added link Link_lidar
Joints:
- removed joint base_joint
- added joint Joint_lidar: type fixed, parent base_link, child Link_lidar, origin xyz=0.109 0 0.0436 rpy=0 0 3.1416, axis 0 0 0
